Commit message: 无头失败，暂存

File: catkin_ws/src/multi_robot_scenario/xacro/p3dx/pioneer3dx.xacro (robot description, xacro)
@@ -1,24 +1,40 @@
 <?xml version="1.0"?>
 <robot xmlns:xacro="http://www.ros.org/wiki/xacro" name="pioneer3dx" >
-  <!-- Import Rviz colors -->
+  <!-- ============================================================ -->
+  <!--                        参数定义                               -->
+  <!-- ============================================================ -->
+  <xacro:arg name="gpu" default="false" />
+  <!-- ============================================================ -->
+  <!--                      通用辅助文件                              -->
+  <!-- ============================================================ -->
   <xacro:include filename="$(find multi_robot_scenario)/xacro/materials.xacro" />
-  <!-- Import robot -->
   <xacro:include filename="$(find multi_robot_scenario)/xacro/p3dx/pioneer3dx_body.xacro"/>
+  <!-- 机器人本体 -->
   <xacro:pioneer3dx_body name="chassis" parent="base_link" meshes="package://gazebo_plugins/test/multi_robot_scenario/meshes/p3dx"/>
-  <!-- Laser -->
-  <xacro:include filename="$(find multi_robot_scenario)/xacro/laser/hokuyo.xacro"/>
-  <xacro:laser name="front_laser" parent="chassis" xyz="0.125 0 0.25" rpy="0 0 0" meshes="package://gazebo_plugins/test/multi_robot_scenario/meshes/laser"/>
-  <!-- GPU Laser
-  <xacro:include filename="$(find multi_robot_scenario)/xacro/laser/hokuyo_gpu.xacro"/>
-  <xacro:laser_gpu name="front_laser" parent="chassis" xyz="0.16 0 0.1" rpy="0 0 0" meshes="package://gazebo_plugins/test/multi_robot_scenario/meshes/laser" />
-    -->
+  <!-- ============================================================ -->
+  <!--            前向单线激光雷达 (Hokuyo) - CPU/GPU 可选            -->
+  <!-- ============================================================ -->
+  <!-- NOTE: Position is IDENTICAL for CPU and GPU versions to ensure consistent training state -->
+  <xacro:if value="$(arg gpu)">
+    <xacro:include filename="$(find multi_robot_scenario)/xacro/laser/hokuyo_gpu.xacro"/>
+    <xacro:laser_gpu name="front_laser" parent="chassis" xyz="0.125 0 0.25" rpy="0 0 0" meshes="package://gazebo_plugins/test/multi_robot_scenario/meshes/laser" />
+  </xacro:if>
+  <xacro:unless value="$(arg gpu)">
+    <xacro:include filename="$(find multi_robot_scenario)/xacro/laser/hokuyo.xacro"/>
+    <xacro:laser name="front_laser" parent="chassis" xyz="0.125 0 0.25" rpy="0 0 0" meshes="package://gazebo_plugins/test/multi_robot_scenario/meshes/laser"/>
+  </xacro:unless>
+  <!-- ============================================================ -->
+  <!--                   3D激光雷达 (Velodyne VLP-16)                -->
+  <!-- ============================================================ -->
+  <xacro:include filename="$(find velodyne_description)/urdf/VLP-16.urdf.xacro"/>
+  <xacro:VLP-16 parent="base_link" name="velodyne" topic="/velodyne_points" hz="10" samples="360" gpu="$(arg gpu)" min_angle="-1.57" max_angle="1.57" min_range="0.1">
+    <origin xyz="0.125 0 0.25" rpy="0 0 0" />
+  </xacro:VLP-16>
+  <!-- ============================================================ -->
+  <!--                        摄像头传感器                            -->
+  <!-- ============================================================ -->
   <xacro:include filename="$(find multi_robot_scenario)/xacro/camera/camera.xacro"/>
   <xacro:cam name="front_camera" parent="chassis" xyz="0.025 0 0.32" rpy="0 0 0" />
   <xacro:include filename="$(find multi_robot_scenario)/xacro/camera/cameraD.xacro"/>
   <xacro:camD name="cameraD" parent="chassis" xyz="0.025 0 0.32" rpy="0 0 0" />
-  <!-- Velodyne -->
-  <xacro:include filename="$(find velodyne_description)/urdf/VLP-16.urdf.xacro"/>
-  <xacro:VLP-16 parent="base_link" name="velodyne" topic="/velodyne_points" hz="10" samples="360" gpu="false" min_angle="-1.57" max_angle="1.57" min_range="0.1">
-    <origin xyz="0.125 0 0.25" rpy="0 0 0" />
-  </xacro:VLP-16>
 </robot>
